File: Electronics/passive-direct-connection/passive-direct-connection/passive-direct-connection.sch (KiCad schematic (older format))
At the start: 10 parts, among them SW1 SW_SPDT, U1 SN75LBC176P

Commit message: added debounce and assigned components
Parts:
- added C1, C2: .1uf, Capacitor_THT:C_Disc_D3.0mm_W1.6mm_P2.50mm, symbol Device:C_Small
- added C3: 10uf, Capacitor_THT:CP_Radial_D4.0mm_P2.00mm, symbol Device:CP_Small
- added D3: 1N4004, Diode_THT:D_DO-15_P2.54mm_Vertical_AnodeUp, symbol Device:D_Small
- added R5: 240, Resistor_THT:R_Axial_DIN0204_L3.6mm_D1.6mm_P2.54mm_Vertical, symbol Device:R_Small
- D1, D2: footprint (none) -> LED_THT:LED_D3.0mm_Clear
- J1: renamed from J?; footprint (none) -> Connector_Phoenix_MC:PhoenixContact_MC_1,5_4-G-3.5_1x04_P3.50mm_Horizontal
- R1, R2, R3, R4: footprint (none) -> Resistor_THT:R_Axial_DIN0204_L3.6mm_D1.6mm_P2.54mm_Vertical
- R6: renamed from R5; footprint (none) -> Resistor_THT:R_Axial_DIN0204_L3.6mm_D1.6mm_P2.54mm_Vertical
- SW1: footprint (none) -> Connector_Phoenix_MC:PhoenixContact_MC_1,5_3-G-3.5_1x03_P3.50mm_Horizontal
Connections:
- net +5V: now also C2.1, C3.1
- net GND: now also C1.1, C2.2, C3.2
- net at D1.2 (A), D2.1 (K), R1.2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: now also D3.2 (A)
- net at R4.2, U1.4 (D): now also C1.2, R5.2
- new net: D3.1 (K), R5.1
- no-connect marks 0 -> 2
Other:
- moved on the sheet: J1, R4, R6, U1

Commit message: set connectors to vertical
Parts:
- J1: footprint Connector_Phoenix_MC:PhoenixContact_MC_1,5_4-G-3.5_1x04_P3.50mm_Horizontal -> Connector_Phoenix_MC:PhoenixContact_MCV_1,5_4-G-3.5_1x04_P3.50mm_Vertical
- SW1: footprint Connector_Phoenix_MC:PhoenixContact_MC_1,5_3-G-3.5_1x03_P3.50mm_Horizontal -> Connector_Phoenix_MC:PhoenixContact_MCV_1,5_3-G-3.5_1x03_P3.50mm_Vertical
Changed lines of the file:
@@
 F 0 "SW1" H 2725 2660 50  0000 C CNN
 F 1 "SW_SPDT" H 2725 2569 50  0000 C CNN
-F 2 "Connector_Phoenix_MC:PhoenixContact_MC_1,5_3-G-3.5_1x03_P3.50mm_Horizontal" H 2725 2375 50  0001 C CNN
+F 2 "Connector_Phoenix_MC:PhoenixContact_MCV_1,5_3-G-3.5_1x03_P3.50mm_Vertical" H 2725 2375 50  0001 C CNN
 F 3 "~" H 2725 2375 50  0001 C CNN
 	1    2725 2375
@@
 F 0 "J1" H 7047 2457 50  0000 R CNN
 F 1 "Conn_01x04_Male" H 7047 2548 50  0000 R CNN
-F 2 "Connector_Phoenix_MC:PhoenixContact_MC_1,5_4-G-3.5_1x04_P3.50mm_Horizontal" H 7075 2575 50  0001 C CNN
+F 2 "Connector_Phoenix_MC:PhoenixContact_MCV_1,5_4-G-3.5_1x04_P3.50mm_Vertical" H 7075 2575 50  0001 C CNN
 F 3 "~" H 7075 2575 50  0001 C CNN
 	1    7075 2575
